Commit message: imported test CAD and added 4 wheels

File: ros2_ws/src/microros_hardware_interface/description/ros2_control/microros_hardware.ros2_control.xacro (robot description, xacro)
@@ -54,6 +54,8 @@
           <plugin>ign_ros2_control/IgnitionSystem</plugin>
         </hardware>
-        <xacro:motor name="left_wheel_joint"/>
-        <xacro:motor name="right_wheel_joint"/>
+        <xacro:motor name="front_left_wheel_joint"/>
+        <xacro:motor name="front_right_wheel_joint"/>
+        <xacro:motor name="back_left_wheel_joint"/>
+        <xacro:motor name="back_right_wheel_joint"/>
       </ros2_control>
       <!-- Setup Gazebo -->

File: ros2_ws/src/microros_hardware_interface/description/urdf/robot.urdf.xacro (robot description, xacro)
@@ -8,4 +8,5 @@
     <!-- Chassis -->
     <link name="${prefix}chassis_link">
+      <!-- COLLISION -->
       <collision>
         <origin xyz="0 0 0" rpy="0 0 ${PI/2}"/>
@@ -14,12 +15,13 @@
         </geometry>
       </collision>
+      <!-- VISUAL -->
       <visual>
-        <origin xyz="0 0 0" rpy="0 0 ${PI/2}"/>
+        <origin xyz="0 0 0" rpy="0 0 0"/>
         <geometry>
           <mesh filename="file://$(find microros_hardware_interface)/description/urdf/assets/chassis/Chassis.dae"/>
         </geometry>
-        <cast_shadows>false</cast_shadows>
-        <material name="grey"/>
+        <cast_shadows>true</cast_shadows>
       </visual>
+      <!-- INERTIAL -->
       <inertial>
         <origin xyz="0 0 0" rpy="0 0 0"/>
@@ -32,10 +34,10 @@
     </link>
     <gazebo reference="chassis_link">
-      <material>Gazebo/Grey</material>
+      <!-- <material>Gazebo/Grey</material> -->
     </gazebo>
     <joint name="${prefix}chassis_joint" type="fixed">
       <parent link="${prefix}base_link"/>
       <child link="${prefix}chassis_link"/>
-      <origin xyz="0 0 ${wheel_radius}" rpy="0 0 ${PI}"/>
+      <origin xyz="0 0 ${wheel_radius}" rpy="0 0 0"/>
       <axis xyz="0 0 1"/>
       <dynamics damping="${damping}"/>
@@ -46,9 +48,10 @@
       <origin xyz="0 0 0" rpy="0 0 0"/>
     </joint>
-    <!--front is positive, left is positive-->
-    <xacro:wheel name="left" x="0" y="0" z="0" front="-1" side="-1"/>
-    <xacro:wheel name="right" x="0" y="0" z="0" front="-1" side="1"/>
-    <xacro:dead_wheel name="left_caster" x="0" y="0" z="0" front="1" side="-1"/>
-    <xacro:dead_wheel name="right_caster" x="0" y="0" z="0" front="1" side="1"/>
+    <!-- Wheels -->
+      <!--front is positive, left is positive-->
+      <xacro:wheel name="front_left" x="${front_left_wheel_x}" y="${front_left_wheel_y}" z="${front_left_wheel_z}" front="1" side="1"/>
+      <xacro:wheel name="front_right" x="${front_right_wheel_x}" y="${front_right_wheel_y}" z="${front_right_wheel_z}" front="1" side="-1"/>
+      <xacro:wheel name="back_left" x="${back_left_wheel_x}" y="${back_left_wheel_y}" z="${back_left_wheel_z}" front="-1" side="1"/>
+      <xacro:wheel name="back_right" x="${back_right_wheel_x}" y="${back_right_wheel_y}" z="${back_right_wheel_z}" front="-1" side="-1"/>
   </xacro:macro>
 </robot>

File: ros2_ws/src/microros_hardware_interface/description/urdf/util/constants.xacro (robot description, xacro)
@@ -1,15 +1,31 @@
 <?xml version="1.0"?>
 <robot xmlns:xacro="http://www.ros.org/wiki/xacro">
-    <xacro:property name="PI" value="3.1415926535897931"/>
-    <xacro:property name="base_mass" value="20" /> <!-- arbitrary value for base mass -->
-    <xacro:property name="base_width" value="0.35" />
-    <xacro:property name="base_length" value="0.50" />
-    <xacro:property name="base_height" value="0.25" />
-    <xacro:property name="wheelbase" value=".2845" />
-    <xacro:property name="wheel_width" value="0.05" />
-    <xacro:property name="wheel_radius" value="0.1" />
-    <xacro:property name="wheel_mass" value="0.5" /> <!-- arbitrary value for wheel mass -->
-    <xacro:property name="friction" value="1"/>
-    <xacro:property name="min_depth" value="0.5"/>
-    <xacro:property name="damping" value="0.001"/>
+    <!-- Physics Constants -->
+        <xacro:property name="PI" value="3.1415926535897931"/>
+        <xacro:property name="friction" value="1"/>
+        <xacro:property name="min_depth" value="0.5"/>
+        <xacro:property name="damping" value="0.001"/>
+    <!-- System Wide Constants -->
+        <xacro:property name="base_mass" value="20" /> <!-- arbitrary value for base mass -->
+        <xacro:property name="base_width" value="0.35" />
+        <xacro:property name="base_length" value="0.50" />
+        <xacro:property name="base_height" value="0.25" />
+    <!-- Mechanism Specific -->
+        <!-- Wheels -->
+            <xacro:property name="wheelbase" value="0.350" />
+            <xacro:property name="wheel_width" value="0.05" />
+            <xacro:property name="wheel_radius" value="0.1" />
+            <xacro:property name="wheel_mass" value="0.5" /> <!-- arbitrary value for wheel mass -->
+            <xacro:property name="front_left_wheel_x" value="0.150"/>
+            <xacro:property name="front_left_wheel_y" value="0.175"/>
+            <xacro:property name="front_left_wheel_z" value="0.00"/>
+            <xacro:property name="front_right_wheel_x" value="0.150"/>
+            <xacro:property name="front_right_wheel_y" value="-0.175"/>
+            <xacro:property name="front_right_wheel_z" value="0.00"/>
+            <xacro:property name="back_left_wheel_x" value="-0.150"/>
+            <xacro:property name="back_left_wheel_y" value="0.175"/>
+            <xacro:property name="back_left_wheel_z" value="0.00"/>
+            <xacro:property name="back_right_wheel_x" value="-0.150"/>
+            <xacro:property name="back_right_wheel_y" value="-0.175"/>
+            <xacro:property name="back_right_wheel_z" value="0.00"/>
 </robot>

File: ros2_ws/src/microros_hardware_interface/description/urdf/util/macros/wheel.xacro (robot description, xacro)
@@ -1,33 +1,36 @@
 <?xml version="1.0"?>
 <robot xmlns:xacro="http://www.ros.org/wiki/xacro">
+    <!-- Macro Header -->
     <xacro:macro name="wheel" params="name x y z front side">
+        <!-- Create Link -->
         <link name="${name}_wheel">
             <!-- COLLISION -->
             <collision>
-            <origin xyz="0 0 0" rpy="0 0 0"/>
-            <geometry>
-                <!-- <mesh filename="file://$(find microros_hardware_interface)/description/urdf/assets/wheel/Wheel.stl"/> -->
-                <sphere radius="${wheel_radius}" />
-            </geometry>
-            <surface>
-                <friction>
-                    <ode>
-                    <mu value="${friction}"/>
-                    <mu2 value="${friction}"/>
-                    <!-- <min_depth value="${min_depth}"/> -->
-                    <!-- <slip1 value="1"/>
-                    <slip2 value="1"/> -->
-                    </ode>
-                    <torsional>
-                    <coefficient>0.0</coefficient>
-                    </torsional>
-                </friction>
-                <contact>
-                    <ode>
-                    <min_depth value="${min_depth}"/>
-                    <!-- <kp>1e15</kp>
-                    <kd>1e13</kd> -->
-                    </ode>
-                </contact>
+                <origin xyz="0 0 0" rpy="0 0 0"/>
+                <geometry>
+                    <!-- <mesh filename="file://$(find microros_hardware_interface)/description/urdf/assets/wheel/Wheel.stl"/> -->
+                    <!-- Collision Calculations are easier with sphere rather than STL -->
+                    <sphere radius="${wheel_radius}" />
+                </geometry>
+                <surface>
+                    <friction>
+                        <ode>
+                        <mu value="${friction}"/>
+                        <mu2 value="${friction}"/>
+                        <!-- <min_depth value="${min_depth}"/> -->
+                        <!-- <slip1 value="1"/> -->
+                        <!-- <slip2 value="1"/> -->
+                        </ode>
+                        <torsional>
+                        <coefficient>0.0</coefficient>
+                        </torsional>
+                    </friction>
+                    <contact>
+                        <ode>
+                        <min_depth value="${min_depth}"/>
+                        <!-- <kp>1e15</kp>
+                        <kd>1e13</kd> -->
+                        </ode>
+                    </contact>
                 </surface>
             </collision>
@@ -51,14 +54,19 @@
             </inertial>
         </link>
+        <!-- Set Gazebo Params -->
         <gazebo reference="${name}_wheel">
-            <material>Gazebo/Black</material>
+            <!-- <material>Gazebo/Black</material> -->
             <mu1 value="10"/>
             <mu2 value="10"/>
         </gazebo>
+        <!-- Create Joint -->
         <joint name="${name}_wheel_joint" type="continuous">
+            <!-- Parent - Child -->
             <parent link="${prefix}chassis_link"/>
             <child link="${name}_wheel"/>
-            <origin xyz="${front * .150} ${side * .175} 0" rpy="${side * -PI/2}  0 0"/>
-            <axis xyz="0 0 ${-side}"/>
+            <!-- Origins and Axis Frames -->
+            <origin xyz="${x} ${y} ${z}" rpy="${side * -PI/2}  0 0"/>
+            <axis xyz="0 0 ${side}"/>
+            <!-- Gazebo Params -->
             <limit effort="1000.0" velocity="100.0"/>
             <dynamics damping="${damping}"/>
