Commit message: seperated chassis into another xacro file

File: ros2_ws/src/microros_hardware_interface/description/urdf/core.urdf.xacro (robot description, xacro)
@@ -5,21 +5,21 @@
   <xacro:arg name="sim_mode" default="false"/>
   <!-- Import Static Files -->
-  <xacro:include filename="$(find microros_hardware_interface)/description/urdf/util/constants.xacro" />
+    <xacro:include filename="$(find microros_hardware_interface)/description/urdf/util/constants.xacro" />
+  <!-- Import Rviz colors -->
+    <xacro:include filename="$(find microros_hardware_interface)/description/urdf/util/materials.xacro" />
   <!-- Import Macros -->
-  <xacro:include filename="$(find microros_hardware_interface)/description/urdf/macros/wheel.xacro" />
-  <!-- <xacro:include filename="$(find microros_hardware_interface)/description/urdf/util/macros/dead_wheel.xacro" /> -->
-  <!-- <xacro:include filename="$(find microros_hardware_interface)/description/urdf/util/macros/camera.xacro" />
-  <xacro:include filename="$(find microros_hardware_interface)/description/urdf/util/macros/depth_camera.xacro" />
-  <xacro:include filename="$(find microros_hardware_interface)/description/urdf/util/macros/imu.xacro" />
-  <xacro:include filename="$(find microros_hardware_interface)/description/urdf/util/macros/lidar.xacro" />
-  <xacro:include filename="$(find microros_hardware_interface)/description/urdf/util/macros/oakd.xacro" /> -->
+    <xacro:include filename="$(find microros_hardware_interface)/description/urdf/macros/wheel.xacro" />
+    <!-- <xacro:include filename="$(find microros_hardware_interface)/description/urdf/util/macros/dead_wheel.xacro" /> -->
+    <!-- <xacro:include filename="$(find microros_hardware_interface)/description/urdf/util/macros/camera.xacro" /> -->
+    <!-- <xacro:include filename="$(find microros_hardware_interface)/description/urdf/util/macros/depth_camera.xacro" /> -->
+    <!-- <xacro:include filename="$(find microros_hardware_interface)/description/urdf/util/macros/imu.xacro" /> -->
+    <!-- <xacro:include filename="$(find microros_hardware_interface)/description/urdf/util/macros/lidar.xacro" /> -->
+    <!-- <xacro:include filename="$(find microros_hardware_interface)/description/urdf/util/macros/oakd.xacro" /> -->
   <!-- Import Robot Description -->
-  <xacro:include filename="$(find microros_hardware_interface)/description/urdf/robot.urdf.xacro" />
-  <!-- Import Rviz colors -->
-  <xacro:include filename="$(find microros_hardware_interface)/description/urdf/util/materials.xacro" />
+    <xacro:include filename="$(find microros_hardware_interface)/description/urdf/robot.urdf.xacro" />
   <!-- Import Hardware Interface -->
-  <xacro:include filename="$(find microros_hardware_interface)/description/ros2_control/microros_hardware.ros2_control.xacro" />
-  <xacro:robot_hardware prefix="$(arg prefix)" />
-  <xacro:micro_system_hardware_ros2_control name="MicroSystemHardware" prefix="$(arg prefix)"/>
+    <xacro:include filename="$(find microros_hardware_interface)/description/ros2_control/microros_hardware.ros2_control.xacro" />
+    <xacro:robot_hardware prefix="$(arg prefix)" />
+    <xacro:micro_system_hardware_ros2_control name="MicroSystemHardware" prefix="$(arg prefix)"/>
   <!-- Hardware Components -->
     <!-- Import Driver Camera -->

File: ros2_ws/src/microros_hardware_interface/description/urdf/robot.urdf.xacro (robot description, xacro)
@@ -6,41 +6,5 @@
     <!-- Base Footprint -->
     <link name="${prefix}base_footprint"/>
-    <!-- Chassis -->
-    <link name="${prefix}chassis_link">
-      <!-- COLLISION -->
-      <collision>
-        <origin xyz="0 0 0" rpy="0 0 ${PI/2}"/>
-        <geometry>
-          <mesh filename="file://$(find microros_hardware_interface)/description/urdf/assets/chassis/Chassis.stl"/>
-        </geometry>
-      </collision>
-      <!-- VISUAL -->
-      <visual>
-        <origin xyz="0 0 0" rpy="0 0 0"/>
-        <geometry>
-          <mesh filename="file://$(find microros_hardware_interface)/description/urdf/assets/chassis/Chassis.dae"/>
-        </geometry>
-        <cast_shadows>true</cast_shadows>
-      </visual>
-      <!-- INERTIAL -->
-      <inertial>
-        <origin xyz="0 0 0" rpy="0 0 0"/>
-        <mass value="${base_mass}"/>
-          <inertia
-            ixx="${0.01952332}" ixy="0.0" ixz="0.0"
-            iyy="${0.01450326}" iyz="${-0.00000016}"
-            izz="${0.02678084}"/>
-        </inertial>
-    </link>
-    <gazebo reference="chassis_link">
-      <!-- <material>Gazebo/Grey</material> -->
-    </gazebo>
-    <joint name="${prefix}chassis_joint" type="fixed">
-      <parent link="${prefix}base_link"/>
-      <child link="${prefix}chassis_link"/>
-      <origin xyz="0 0 ${wheel_radius}" rpy="0 0 0"/>
-      <axis xyz="0 0 1"/>
-      <dynamics damping="${damping}"/>
-    </joint>
+    <!-- Base Link - Base Footprint -->
     <joint name="${prefix}base_footprint_joint" type="fixed">
       <parent link="${prefix}base_link"/>
@@ -48,4 +12,6 @@
       <origin xyz="0 0 0" rpy="0 0 0"/>
     </joint>
+    <!-- Chassis -->
+    <xacro:include filename="$(find microros_hardware_interface)/description/urdf/components/chassis.xacro" />
     <!-- Wheels -->
       <!--front is positive, left is positive-->
